Commit message: fix: robot model working on gazebo and camera

File: Intro_ROS/robot_differential_sena/urdf/robot_differential_sena.urdf (robot description, URDF)
Before this commit: robot robot_differential_sena, 5 links, 4 joints
Links:
- removed link Camara_Link
- removed link Lidar_Link
- removed link RuedaDerecha_Link
- removed link RuedaIzquierda_Link
- added link Camara_link, mass 0; collision mesh filename=package://robot_differential_sena/meshes/Camara_link.STL; visual mesh filename=package://robot_differential_sena/meshes/Camara_link.STL
- added link Lidar_link, mass 0; collision mesh filename=package://robot_differential_sena/meshes/Lidar_link.STL; visual mesh filename=package://robot_differential_sena/meshes/Lidar_link.STL
- added link RuedaDerecha_link, mass 0.033874; collision mesh filename=package://robot_differential_sena/meshes/RuedaDerecha_link.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; visual mesh filename=package://robot_differential_sena/meshes/RuedaDerecha_link.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
- added link RuedaIzquierda_link, mass 0.033874; collision mesh filename=package://robot_differential_sena/meshes/RuedaIzquierda_lin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; visual mesh filename=package://robot_differential_sena/meshes/RuedaIzquierda_lin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
Joints:
- removed joint Camara_Joint
- removed joint Lidar_Joint
- removed joint RuedaDerecha_Joint
- removed joint RuedaIzquierda_Joint
- added joint Camara_joint: type fixed, parent base_link, child Camara_link, origin xyz=-0.0019769 0.09428 0.1277 rpy=-1.5708 0 0.01852, axis 0 0 0
- added joint Lidar_joint: type fixed, parent base_link, child Lidar_link, origin xyz=0 0.07275 0.2396 rpy=-1.5708 0 -1.5708, axis 0 0 0
- added joint RuedaDerecha_joint: type continuous, parent base_link, child RuedaDerecha_link, origin xyz=0.08245 0.056047 0.0195 rpy=-1.8147 0 3.1416, axis 1 0 0
- added joint RuedaIzquierda_joint: type continuous, parent base_link, child RuedaIzquierda_link, origin xyz=-0.08245 0.056047 0.0195 rpy=2.6278 0 0, axis -1 0 0
